File: oled-bmp280-touch.kicad_pcb (KiCad board)
At the start: 2 copper layers, 50 x 51.7 mm, 8 parts, among them J1 TEENSY-LC

Commit message: update layout
Parts:
- added G***: LOGO, teensy-big-oled:oshpark-silk-25dpi, B.Cu at (96.8, 107.3)
- added G***: LOGO, teensy-big-oled:osh-park-logo-300dpi-normal-silk, F.Cu at (84.1, 104.6)
- added REF**: Symbol_OSHW-Logo_SilkScreen, CHIP-DIPs:Symbol_OSHW-Logo_SilkScreen, F.Cu at (115.3, 103.4)
Other:
- outline, holes or cut-outs redrawn
- board text added: "DREW FUSTINI"
- board text added: "drew@oshpark.com"
